File: hardware/Power.kicad_sch (KiCad schematic)
At the start: 15 parts

Commit message: hw: update
Parts:
- added C5, C6, C7: 10uf, Capacitor_SMD:C_1206_3216Metric, symbol Device:C
- added J3: POWER, misc:PinHeader_1x02_P2.54mm_Vertical, symbol Connector_Generic:Conn_01x02
- C8: renamed from C?; footprint Capacitor_SMD:C_0603_1608Metric -> Capacitor_SMD:C_1206_3216Metric
- D5: renamed from D?; footprint (none) -> LED_SMD:LED_0603_1608Metric
- L1: value 68uH -> 22uH; footprint Inductor_SMD:L_Taiyo-Yuden_NR-60xx_HandSoldering -> Inductor_SMD:L_Taiyo-Yuden_NR-40xx
- U2: renamed from U?; symbol mylib:TX4137 -> misc:TX4137
- gave numbers to parts that had none: 11
Connections:
- net GND: now also C5.1, C6.1, C7.1, J3.1 (Pin_1)
- net V_SUPPLY: now also C5.2, C6.2, C7.2, J3.2 (Pin_2)
Other:
- moved on the sheet: C8
