File: hardware/solar_tracer.kicad_sch (KiCad schematic)
At the start: 25 parts

Commit message: hw: update
Parts:
- removed C? (x4): 100nf, Capacitor_SMD:C_0402_1005Metric, symbol Device:C
- removed C? (x2): 10uf, Capacitor_SMD:C_0603_1608Metric, symbol Device:C
- removed J?: MOTY, misc:PinHeader_1x02_P2.54mm_Vertical, symbol Connector_Generic:Conn_01x02
- removed J?: IMU, symbol Connector_Generic:Conn_01x04
- removed J?: MOTX, misc:PinHeader_1x02_P2.54mm_Vertical, symbol Connector_Generic:Conn_01x02
- removed R? (x2): 4.7k, Resistor_SMD:R_0402_1005Metric, symbol Device:R
- removed R?: 10k, Resistor_SMD:R_0402_1005Metric, symbol Device:R
- removed U?: ESP32-C6-WROOM-1, Espressif:ESP32-C3-WROOM-02U, symbol Espressif:ESP32-C6-WROOM-1
- removed U? (x2): AT8236, Package_SO:SOIC-8-1EP_3.9x4.9mm_P1.27mm_EP2.29x3mm, symbol misc:AT8236
- removed U?: JY901x, symbol misc:JY901x
- added D1: GREEN, LED_SMD:LED_0603_1608Metric, symbol Device:LED
- added H1, H2, H3, H4: MountingHole_Pad, MountingHole:MountingHole_3.2mm_M3_Pad_Via, symbol Mechanical:MountingHole_Pad
- added R2: 4.7k, Resistor_SMD:R_0402_1005Metric, symbol Device:R
- added U1: ESP32-S3-WROOM-1, Espressif:ESP32-S3-WROOM-1, symbol Espressif:ESP32-S3-WROOM-1
- D2: renamed from D?; footprint (none) -> LED_SMD:LED_0603_1608Metric
- J1: renamed from J?; footprint (none) -> Connector_PinHeader_2.54mm:PinHeader_1x06_P2.54mm_Vertical
- J2: renamed from J?; footprint (none) -> misc:PinHeader_1x04_P2.54mm_Vertical
- R3: renamed from R?; value 1k -> 4.7k
- gave numbers to parts that had none: 5
Connections:
- net BOOT: now also J1.3 (Pin_3), U1.27 (GPIO0/BOOT); no longer J1.5 (Pin_5)
- net EN: now also U1.3 (EN)
- net GND: now also J2.3 (Pin_3), D1.1 (K), H1.1, H2.1, H3.1, H4.1, U1.1 (GND), U1.40 (GND), U1.41 (GND); no longer J2.2 (Pin_2)
- net GPS_RX: now also J2.1 (Pin_1), U1.28 (SPIIO6/GPIO35/FSPID/SUBSPID); no longer J2.4 (Pin_4)
- net GPS_TX: now also J2.2 (Pin_2), U1.29 (SPIIO7/GPIO36/FSPICLK/SUBSPICLK); no longer J2.3 (Pin_3)
- net RX0: now also J1.4 (Pin_4), U1.36 (U0RXD/GPIO44/CLK_OUT2); no longer J1.3 (Pin_3)
- net TX0: now also J1.5 (Pin_5), U1.37 (U0TXD/GPIO43/CLK_OUT1); no longer J1.4 (Pin_4)
- net VCC: now also J2.4 (Pin_4), U1.2 (3V3); no longer J2.1 (Pin_1)
- net power/ADC_POWER: now also U1.39 (GPIO1/TOUCH1/ADC1_CH0)
- net at R3.1: now also U1.35 (MTMS/GPIO42)
- new net: R2.1, U1.34 (MTDI/GPIO41/CLK_OUT1)
- new net: D1.2 (A), R2.2
- new net IMU_SCL: U1.30 (SPIDQS/GPIO37/FSPIQ/SUBSPIQ)
- new net IMU_SDA: U1.31 (GPIO38/FSPIWP/SUBSPIWP)
- new net MOTY_IN1: U1.8 (GPIO15/U0RTS/ADC2_CH4/XTAL_32K_P)
- new net MOTY_IN2: U1.9 (GPIO16/U0CTS/ADC2_CH5/XTAL_32K_N)
- new net motor/MOTX_ENCA: U1.5 (GPIO5/TOUCH5/ADC1_CH4)
- new net motor/MOTX_ENCB: U1.4 (GPIO4/TOUCH4/ADC1_CH3)
- new net motor/MOTX_IN1: U1.6 (GPIO6/TOUCH6/ADC1_CH5)
- new net motor/MOTX_IN2: U1.7 (GPIO7/TOUCH7/ADC1_CH6)
- new net motor/MOTY_ENCA: U1.11 (GPIO18/U1RXD/ADC2_CH7/CLK_OUT3)
- new net motor/MOTY_ENCB: U1.10 (GPIO17/U1TXD/ADC2_CH6)
- no-connect marks 6 -> 20
Other:
- added sheet imu (imu.kicad_sch)
- added sheet motor (motor.kicad_sch)
- note added: "Mounting Holes"
- moved on the sheet: C1, C2, C3, D2, R1, R3
